Commit message: Tweak some parameters. Add effort_controller and a new extending link

File: urdf/bookshelf_robot.urdf.xacro (robot description, xacro)
@@ -18,13 +18,13 @@
   <xacro:property name="wheel_length" value="0.08" />
   <xacro:property name="wheel_radius" value="0.2" />
-  <xacro:property name="wheel_mass" value="1" />
+  <xacro:property name="wheel_mass" value="0.2" />
   <!-- Caster leg link propersties -->
   <xacro:property name="caster_leg_length" value="0.05" />
   <xacro:property name="caster_leg_width" value="0.05" />
-  <xacro:property name="caster_leg_height" value="0.08" />
-  <xacro:property name="caster_leg_mass" value="0.3"/>
+  <xacro:property name="caster_leg_height" value="0.1" />
+  <xacro:property name="caster_leg_mass" value="0.1"/>
   <!-- Caster leg link properties -->
   <xacro:property name="caster_radius" value="0.04"/>
-  <xacro:property name="caster_mass" value="0.3"/>
+  <xacro:property name="caster_mass" value="0.1"/>
   <!-- ############ -->
   <!-- Robotic arm  -->
@@ -33,37 +33,42 @@
   <xacro:property name="arm_base_radius" value="0.20"/>
   <xacro:property name="arm_base_length" value="0.05"/>
-  <xacro:property name="arm_base_mass" value="0.5" />
+  <xacro:property name="arm_base_mass" value="1" />
   <!-- Torso properties -->
   <xacro:property name="torso_radius" value="0.05"/>
-  <xacro:property name="torso_length" value="1"/>
-  <xacro:property name="torso_mass" value="0.5" />
+  <xacro:property name="torso_length" value="1.2"/>
+  <xacro:property name="torso_mass" value="0.25" />
   <!-- Arm properties -->
   <xacro:property name="arm_radius" value="0.05"/>
-  <xacro:property name="arm_length" value="0.7"/>
-  <xacro:property name="arm_mass" value="0.25" />
+  <xacro:property name="arm_length" value="0.4"/>
+  <xacro:property name="arm_mass" value="0.1" />
+  <!-- Elbow properties -->
+  <xacro:property name="elbow_radius" value="0.05"/>
+  <xacro:property name="elbow_length" value="0.7"/>
+  <xacro:property name="elbow_mass" value="0.1" />
   <!-- Hand properties -->
   <!-- Hand base -->
   <xacro:property name="hand_base_length" value="0.08" />
   <xacro:property name="hand_base_radius" value="0.01" />
-  <xacro:property name="hand_base_mass" value="0.1"/>
+  <xacro:property name="hand_base_mass" value="0.05"/>
   <!-- Hand palm -->
   <xacro:property name="hand_palm_length" value="0.2" />
   <xacro:property name="hand_palm_width" value="0.01" />
   <xacro:property name="hand_palm_height" value="0.05" />
-  <xacro:property name="hand_palm_mass" value="0.1"/>
+  <xacro:property name="hand_palm_mass" value="0.08"/>
   <!-- Hand finger -->
   <xacro:property name="hand_finger_length" value="0.2" />
   <xacro:property name="hand_finger_width" value="0.01" />
-  <xacro:property name="hand_finger_height" value="0.025" />
-  <xacro:property name="hand_finger_mass" value="0.1"/>
+  <xacro:property name="hand_finger_height" value="0.06" />
+  <xacro:property name="hand_finger_mass" value="0.05"/>
   <!-- ########################## -->
   <!-- Mobile base implementation -->
   <!-- ########################## -->
-  <!-- <link name="footprint" />
+  <link name="footprint">
+  </link>
   <joint name="base_joint" type="fixed">
     <parent link="footprint"/>
     <child link="chassis"/>
-    <origin rpy="0 0 0" xyz="0 0 0"/>
-  </joint> -->
+    <origin rpy="0 0 0" xyz="0 0 ${wheel_radius}"/>
+  </joint>
   <link name="chassis">
     <visual>
@@ -127,5 +132,5 @@
     <parent link="chassis"/>
     <child link="right_wheel"/>
-    <origin rpy="${-PI/2} 0 0" xyz="${-chassis_length/4} ${+chassis_width/2+wheel_length/2} 0"/>
+    <origin rpy="${-PI/2} 0 0" xyz="${-chassis_length/4}  ${+chassis_width/2+wheel_length/2} 0"/>
   </joint>
   <link name="caster_leg">
@@ -179,6 +184,10 @@
       <rightJoint>right_wheel_joint</rightJoint>
       <robotBaseFrame>chassis</robotBaseFrame>
-      <wheelSeparation>${chassis_width}</wheelSeparation>
+      <wheelSeparation>${chassis_width-wheel_length}</wheelSeparation>
       <wheelDiameter>${2*wheel_radius}</wheelDiameter>
+      <odometryTopic>odom</odometryTopic>
+      <odometryFrame>odom</odometryFrame>
+      <publishWheelTF>true</publishWheelTF>
+      <rosDebugLevel>na</rosDebugLevel>
       <publishWheelJointState>true</publishWheelJointState>
     </plugin>
@@ -238,7 +247,9 @@
         <cylinder length="${arm_length}" radius="${arm_radius}"/>
       </geometry>
+      <origin rpy="0 0 0" xyz="0 0 ${-arm_length/2}"/>
       <material name="orange"/>
     </visual>
     <collision>
+      <origin rpy="0 0 0" xyz="0 0 ${-arm_length/2}"/>
       <geometry>
         <cylinder length="${arm_length}" radius="${arm_radius}"/>
@@ -246,4 +257,5 @@
     </collision>
     <inertial>
+      <origin rpy="0 0 0" xyz="0 0 ${-arm_length/2}"/>
       <mass value="${arm_mass}"/>
       <cylinder_inertia m="${arm_mass}" r="${arm_length}" h="${arm_radius}"/>
@@ -253,7 +265,34 @@
     <parent link="torso"/>
     <child link="arm"/>
-    <origin rpy="0 ${-PI/2} 0" xyz="${arm_length/2} 0 ${-torso_length/2}"/>
+    <origin rpy="0 ${-PI/2} 0" xyz="0 ${-2*arm_radius} ${-torso_length/2}"/>
     <axis xyz="1 0 0"/>
-    <limit effort="4" lower="0" upper="0.9" velocity="0.15" />
+    <limit effort="10.0" lower="0.0" upper="0.9" velocity="10" />
+  </joint>
+  <link name="elbow">
+    <visual>
+      <geometry>
+        <cylinder length="${elbow_length}" radius="${elbow_radius}"/>
+      </geometry>
+      <origin rpy="0 0 0" xyz="0 0 ${-elbow_length/2}"/>
+      <material name="orange"/>
+    </visual>
+    <collision>
+      <origin rpy="0 0 0" xyz="0 0 ${-elbow_length/2}"/>
+      <geometry>
+        <cylinder length="${elbow_length}" radius="${elbow_radius}"/>
+      </geometry>
+    </collision>
+    <inertial>
+      <origin rpy="0 0 0" xyz="0 0 ${-arm_length/2}"/>
+      <mass value="${elbow_mass}"/>
+      <cylinder_inertia m="${elbow_mass}" r="${elbow_length}" h="${elbow_radius}"/>
+    </inertial>
+  </link>
+  <joint name="elbow_joint" type="prismatic">
+    <parent link="arm"/>
+    <child link="elbow"/>
+    <origin rpy="0 0 0" xyz="0 ${2*arm_radius} ${-arm_length/2}"/>
+    <axis xyz="0 0 1"/>
+    <limit effort="10.0" lower="0.0" upper="0.15" velocity="10" />
   </joint>
   <link name="hand_base">
@@ -278,8 +317,8 @@
   </link>
   <joint name="wrist_joint" type="revolute">
-    <parent link="arm"/>
+    <parent link="elbow"/>
     <child link="hand_base"/>
     <axis xyz="0 1 0"/>
-    <origin rpy="0 0 0" xyz="0 0 ${-arm_length/2}-{hand_base_length/2}"/>
+    <origin rpy="0 0 0" xyz="0 0 ${-elbow_length}-{hand_base_length/2}"/>
     <limit effort="1" lower="${-PI/2}" upper="${PI/2}" velocity="0.15" />
   </joint>
@@ -332,5 +371,5 @@
     <origin rpy="0 0 ${PI/2}" xyz="${-hand_palm_length/2} 0 0"/>
     <axis xyz="0 -1 0"/>
-    <limit effort="0.5" lower="0" upper="0.05" velocity="0.15" />
+    <limit effort="10" lower="0" upper="0.05" velocity="0.4" />
   </joint>
   <link name="hand_right_finger">
@@ -359,13 +398,13 @@
     <origin rpy="0 0 ${PI/2}" xyz="${hand_palm_length/2} 0 0"/>
     <axis xyz="0 1 0"/>
-    <limit effort="0.5" lower="0" upper="0.05" velocity="0.15" />
+    <limit effort="10" lower="0" upper="0.05" velocity="0.4" />
   </joint>
   <transmission name="tran0">
     <type>transmission_interface/SimpleTransmission</type>
     <joint name="hip_joint">
-      <hardwareInterface>PositionJointInterface</hardwareInterface>
+      <hardwareInterface>hardware_interface/PositionJointInterface</hardwareInterface>
     </joint>
     <actuator name="motor0">
-      <hardwareInterface>PositionJointInterface</hardwareInterface>
+      <hardwareInterface>hardware_interface/PositionJointInterface</hardwareInterface>
       <mechanicalReduction>1</mechanicalReduction>
     </actuator>
@@ -374,8 +413,18 @@
     <type>transmission_interface/SimpleTransmission</type>
     <joint name="shoulder_joint">
-      <hardwareInterface>PositionJointInterface</hardwareInterface>
+      <hardwareInterface>hardware_interface/EffortJointInterface</hardwareInterface>
     </joint>
     <actuator name="motor1">
-      <hardwareInterface>PositionJointInterface</hardwareInterface>
+      <hardwareInterface>hardware_interface/EffortJointInterface</hardwareInterface>
+      <mechanicalReduction>1</mechanicalReduction>
+    </actuator>
+  </transmission>
+  <transmission name="tran5">
+    <type>transmission_interface/SimpleTransmission</type>
+    <joint name="elbow_joint">
+      <hardwareInterface>hardware_interface/EffortJointInterface</hardwareInterface>
+    </joint>
+    <actuator name="motor5">
+      <hardwareInterface>hardware_interface/EffortJointInterface</hardwareInterface>
       <mechanicalReduction>1</mechanicalReduction>
     </actuator>
@@ -384,8 +433,8 @@
     <type>transmission_interface/SimpleTransmission</type>
     <joint name="wrist_joint">
-      <hardwareInterface>PositionJointInterface</hardwareInterface>
+      <hardwareInterface>hardware_interface/PositionJointInterface</hardwareInterface>
     </joint>
     <actuator name="motor2">
-      <hardwareInterface>PositionJointInterface</hardwareInterface>
+      <hardwareInterface>hardware_interface/PositionJointInterface</hardwareInterface>
       <mechanicalReduction>1</mechanicalReduction>
     </actuator>
@@ -394,8 +443,8 @@
     <type>transmission_interface/SimpleTransmission</type>
     <joint name="left_finger_joint">
-      <hardwareInterface>PositionJointInterface</hardwareInterface>
+      <hardwareInterface>hardware_interface/EffortJointInterface</hardwareInterface>
     </joint>
     <actuator name="motor3">
-      <hardwareInterface>PositionJointInterface</hardwareInterface>
+      <hardwareInterface>hardware_interface/EffortJointInterface</hardwareInterface>
       <mechanicalReduction>1</mechanicalReduction>
     </actuator>
@@ -404,8 +453,8 @@
     <type>transmission_interface/SimpleTransmission</type>
     <joint name="right_finger_joint">
-      <hardwareInterface>PositionJointInterface</hardwareInterface>
+      <hardwareInterface>hardware_interface/EffortJointInterface</hardwareInterface>
     </joint>
     <actuator name="motor4">
-      <hardwareInterface>PositionJointInterface</hardwareInterface>
+      <hardwareInterface>hardware_interface/EffortJointInterface</hardwareInterface>
       <mechanicalReduction>1</mechanicalReduction>
     </actuator>

Commit message: PID seems ok. Teleop with Xbox Joystick.

File: urdf/bookshelf_robot.urdf.xacro (robot description, xacro)
@@ -40,6 +40,6 @@
   <!-- Arm properties -->
   <xacro:property name="arm_radius" value="0.05"/>
-  <xacro:property name="arm_length" value="0.4"/>
-  <xacro:property name="arm_mass" value="0.1" />
+  <xacro:property name="arm_length" value="0.5"/>
+  <xacro:property name="arm_mass" value="0.05" />
   <!-- Elbow properties -->
   <xacro:property name="elbow_radius" value="0.05"/>
@@ -188,5 +188,5 @@
       <odometryTopic>odom</odometryTopic>
       <odometryFrame>odom</odometryFrame>
-      <publishWheelTF>true</publishWheelTF>
+      <publishWheelTF>false</publishWheelTF>
       <rosDebugLevel>na</rosDebugLevel>
       <publishWheelJointState>true</publishWheelJointState>
@@ -240,5 +240,5 @@
     <child link="torso"/>
     <origin rpy="0 0 0" xyz="0.0 0.0 ${-torso_length/2}"/>
-    <limit effort="1" velocity="0.15" />
+    <!-- <limit effort="1" velocity="0.15" /> -->
   </joint>
   <link name="arm">
@@ -267,5 +267,5 @@
     <origin rpy="0 ${-PI/2} 0" xyz="0 ${-2*arm_radius} ${-torso_length/2}"/>
     <axis xyz="1 0 0"/>
-    <limit effort="10.0" lower="0.0" upper="0.9" velocity="10" />
+    <limit effort="100.0" lower="0.0" upper="1.1" velocity="1" />
   </joint>
   <link name="elbow">
@@ -294,5 +294,5 @@
     <origin rpy="0 0 0" xyz="0 ${2*arm_radius} ${-arm_length/2}"/>
     <axis xyz="0 0 1"/>
-    <limit effort="10.0" lower="0.0" upper="0.15" velocity="10" />
+    <limit effort="10.0" lower="0.0" upper="0.25" velocity="10" />
   </joint>
   <link name="hand_base">
@@ -371,5 +371,5 @@
     <origin rpy="0 0 ${PI/2}" xyz="${-hand_palm_length/2} 0 0"/>
     <axis xyz="0 -1 0"/>
-    <limit effort="10" lower="0" upper="0.05" velocity="0.4" />
+    <limit effort="50" lower="0" upper="0.05" velocity="0.4" />
   </joint>
   <link name="hand_right_finger">
@@ -398,5 +398,5 @@
     <origin rpy="0 0 ${PI/2}" xyz="${hand_palm_length/2} 0 0"/>
     <axis xyz="0 1 0"/>
-    <limit effort="10" lower="0" upper="0.05" velocity="0.4" />
+    <limit effort="50" lower="0" upper="0.05" velocity="0.4" />
   </joint>
   <transmission name="tran0">
@@ -465,5 +465,5 @@
   <gazebo>
     <plugin name="joint_state_publisher" filename="libgazebo_ros_joint_state_publisher.so">
-      <jointName>hip_joint, shoulder_joint, wrist_joint, left_finger_joint, right_finger_joint </jointName>
+      <jointName>hip_joint, shoulder_joint, elbow_joint, wrist_joint, left_finger_joint, right_finger_joint </jointName>
     </plugin>
 </gazebo>

Commit message: Joints controller by joy messages

File: urdf/bookshelf_robot.urdf.xacro (robot description, xacro)
@@ -267,5 +267,5 @@
     <origin rpy="0 ${-PI/2} 0" xyz="0 ${-2*arm_radius} ${-torso_length/2}"/>
     <axis xyz="1 0 0"/>
-    <limit effort="100.0" lower="0.0" upper="1.1" velocity="1" />
+    <limit effort="100.0" lower="-0.1" upper="1.1" velocity="1" />
   </joint>
   <link name="elbow">

Commit message: Implement head camera.

File: urdf/bookshelf_robot.urdf.xacro (robot description, xacro)
@@ -61,4 +61,7 @@
   <xacro:property name="hand_finger_height" value="0.06" />
   <xacro:property name="hand_finger_mass" value="0.05"/>
+  <!-- Camera -->
+  <xacro:property name="camera_dimensions" value="0.05" />
+  <xacro:property name="camera_mass" value="0.01" />
   <!-- ########################## -->
   <!-- Mobile base implementation -->
@@ -267,5 +270,5 @@
     <origin rpy="0 ${-PI/2} 0" xyz="0 ${-2*arm_radius} ${-torso_length/2}"/>
     <axis xyz="1 0 0"/>
-    <limit effort="100.0" lower="-0.1" upper="1.1" velocity="1" />
+    <limit effort="100.0" lower="0.0" upper="1.1" velocity="1" />
   </joint>
   <link name="elbow">
@@ -399,4 +402,29 @@
     <axis xyz="0 1 0"/>
     <limit effort="50" lower="0" upper="0.05" velocity="0.4" />
+  </joint>
+  <!-- Camera -->
+  <link name="camera_link">
+    <collision>
+      <geometry>
+      <box size="${camera_dimensions} ${camera_dimensions} ${camera_dimensions}"/>
+      </geometry>
+    </collision>
+    <visual>
+      <origin xyz="0 0 0" rpy="0 0 0"/>
+      <geometry>
+      <box size="${camera_dimensions} ${camera_dimensions} ${camera_dimensions}"/>
+      </geometry>
+      <material name="white"/>
+    </visual>
+    <inertial>
+      <mass value="${camera_mass}"/>
+      <box_inertia m="${camera_mass}" x="${camera_dimensions}" y="${camera_dimensions}" z="${camera_dimensions}"/>
+    </inertial>
+  </link>
+  <joint name="camera_joint" type="fixed">
+    <axis xyz="0 1 0" />
+    <origin xyz="0 0 ${-torso_length/2}" rpy="0 0 0"/>
+    <parent link="torso"/>
+    <child link="camera_link"/>
   </joint>
   <transmission name="tran0">
@@ -467,4 +495,4 @@
       <jointName>hip_joint, shoulder_joint, elbow_joint, wrist_joint, left_finger_joint, right_finger_joint </jointName>
     </plugin>
-</gazebo>
+  </gazebo>
 </robot>

Commit message: Change top camera to arm camera. Planning to add a LaserScanner

File: urdf/bookshelf_robot.urdf.xacro (robot description, xacro)
@@ -411,5 +411,5 @@
     </collision>
     <visual>
-      <origin xyz="0 0 0" rpy="0 0 0"/>
+      <origin xyz="${-camera_dimensions/2} 0 0" rpy="0 0 0"/>
       <geometry>
       <box size="${camera_dimensions} ${camera_dimensions} ${camera_dimensions}"/>
@@ -424,6 +424,6 @@
   <joint name="camera_joint" type="fixed">
     <axis xyz="0 1 0" />
-    <origin xyz="0 0 ${-torso_length/2}" rpy="0 0 0"/>
-    <parent link="torso"/>
+    <origin xyz="${-elbow_radius} 0 ${-elbow_length}" rpy="${PI} ${PI/2} 0"/>
+    <parent link="elbow"/>
     <child link="camera_link"/>
   </joint>

Commit message: Add a lidar sensor

File: urdf/bookshelf_robot.urdf.xacro (robot description, xacro)
@@ -64,4 +64,12 @@
   <xacro:property name="camera_dimensions" value="0.05" />
   <xacro:property name="camera_mass" value="0.01" />
+  <!-- Laser Scanner -->
+  <xacro:property name="lidar_base_length" value="0.04" />
+  <xacro:property name="lidar_base_radius" value="0.01" />
+  <xacro:property name="lidar_base_mass" value="0.05"/>
+  <xacro:property name="lidar_length" value="0.05" />
+  <xacro:property name="lidar_width" value="0.05" />
+  <xacro:property name="lidar_height" value="0.05" />
+  <xacro:property name="lidar_mass" value="0.1"/>
   <!-- ########################## -->
   <!-- Mobile base implementation -->
@@ -423,8 +431,56 @@
   </link>
   <joint name="camera_joint" type="fixed">
-    <axis xyz="0 1 0" />
     <origin xyz="${-elbow_radius} 0 ${-elbow_length}" rpy="${PI} ${PI/2} 0"/>
     <parent link="elbow"/>
     <child link="camera_link"/>
+  </joint>
+  <!-- Laser Scanner -->
+<link name="lidar_base">
+    <visual>
+      <geometry>
+        <cylinder length="${lidar_base_length}" radius="${lidar_base_radius}"/>
+      </geometry>
+      <origin rpy="0 0 0" xyz="0 0 ${lidar_base_length/2}"/>
+      <material name="white"/>
+    </visual>
+    <collision>
+      <geometry>
+        <cylinder length="${lidar_base_length}" radius="${lidar_base_radius}"/>
+      </geometry>
+      <origin rpy="0 0 0" xyz="0 0 0"/>
+    </collision>
+    <inertial>
+      <mass value="${lidar_base_mass}"/>
+      <cylinder_inertia m="${lidar_base_mass}" r="${lidar_base_radius}" h="${lidar_base_length}"/>
+      <origin rpy="0 0 0" xyz="0 0 0"/>
+    </inertial>
+  </link>
+  <joint name="base_lidar_joint" type="fixed">
+    <origin xyz="${chassis_length/3} 0 ${chassis_height/2}" rpy="0 0 0"/>
+    <parent link="chassis"/>
+    <child link="lidar_base"/>
+  </joint>
+  <link name="lidar_link">
+    <visual>
+      <geometry>
+        <box size="${lidar_length} ${lidar_width} ${lidar_height}"/>
+      </geometry>
+      <origin xyz="0 0 0" rpy="0 0 0"/>
+      <material name="white"/>
+    </visual>
+    <collision>
+      <geometry>
+        <box size="${lidar_length} ${lidar_width} ${lidar_height}"/>
+      </geometry>
+    </collision>
+    <inertial>
+      <mass value="${chassis_mass}"/>
+      <box_inertia m="${lidar_mass}" x="${lidar_length}" y="${lidar_width}" z="${lidar_height}"/>
+    </inertial>
+  </link>
+  <joint name="lidar_joint" type="fixed">
+    <origin xyz="0 0 ${lidar_base_length}" rpy="0 0 0"/>
+    <parent link="lidar_base"/>
+    <child link="lidar_link"/>
   </joint>
   <transmission name="tran0">

Commit message: Latest OK version. A lot of changes, didn't keep track...

File: urdf/bookshelf_robot.urdf.xacro (robot description, xacro)
@@ -278,5 +278,5 @@
     <origin rpy="0 ${-PI/2} 0" xyz="0 ${-2*arm_radius} ${-torso_length/2}"/>
     <axis xyz="1 0 0"/>
-    <limit effort="100.0" lower="0.0" upper="1.1" velocity="1" />
+    <limit effort="100.0" lower="0.0" upper="1.1" velocity="100" />
   </joint>
   <link name="elbow">
@@ -362,4 +362,29 @@
         <box size="${hand_finger_length} ${hand_finger_width} ${hand_finger_height}"/>
       </geometry>
+      <origin rpy="0 0 0" xyz="${hand_finger_length/2} 0 0"/>
+      <material name="blue"/>
+    </visual>
+    <collision>
+      <geometry>
+        <box size="${hand_finger_length} ${hand_finger_width} ${hand_finger_height}"/>
+      </geometry>
+      <origin rpy="0 0 0" xyz="${hand_finger_length/2} 0 0"/>
+    </collision>
+    <inertial>
+      <mass value="${hand_palm_mass}"/>
+      <box_inertia m="${hand_palm_mass}" x="${hand_finger_length}" y="${hand_finger_width}" z="${hand_finger_height}"/>
+      <origin rpy="0 0 0" xyz="${hand_finger_length/2} 0 0"/>
+    </inertial>
+  </link>
+  <joint name="left_finger_joint" type="fixed">
+    <parent link="hand_right_finger"/>
+    <child link="hand_left_finger"/>
+    <origin rpy="0 0 ${PI/2}" xyz="${-hand_palm_length} 0 0"/>
+  </joint>
+  <link name="hand_right_finger">
+    <visual>
+      <geometry>
+        <box size="${hand_finger_length} ${hand_finger_width} ${hand_finger_height}"/>
+      </geometry>
       <origin rpy="0 0 0" xyz="${-hand_finger_length/2} 0 0"/>
       <material name="blue"/>
@@ -377,37 +402,8 @@
     </inertial>
   </link>
-  <joint name="left_finger_joint" type="prismatic">
-    <parent link="hand_palm"/>
-    <child link="hand_left_finger"/>
-    <origin rpy="0 0 ${PI/2}" xyz="${-hand_palm_length/2} 0 0"/>
-    <axis xyz="0 -1 0"/>
-    <limit effort="50" lower="0" upper="0.05" velocity="0.4" />
-  </joint>
-  <link name="hand_right_finger">
-    <visual>
-      <geometry>
-        <box size="${hand_finger_length} ${hand_finger_width} ${hand_finger_height}"/>
-      </geometry>
-      <origin rpy="0 0 0" xyz="${-hand_finger_length/2} 0 0"/>
-      <material name="blue"/>
-    </visual>
-    <collision>
-      <geometry>
-        <box size="${hand_finger_length} ${hand_finger_width} ${hand_finger_height}"/>
-      </geometry>
-      <origin rpy="0 0 0" xyz="${-hand_finger_length/2} 0 0"/>
-    </collision>
-    <inertial>
-      <mass value="${hand_palm_mass}"/>
-      <box_inertia m="${hand_palm_mass}" x="${hand_finger_length}" y="${hand_finger_width}" z="${hand_finger_height}"/>
-      <origin rpy="0 0 0" xyz="${-hand_finger_length/2} 0 0"/>
-    </inertial>
-  </link>
-  <joint name="right_finger_joint" type="prismatic">
+  <joint name="right_finger_joint" type="fixed">
     <parent link="hand_palm"/>
     <child link="hand_right_finger"/>
     <origin rpy="0 0 ${PI/2}" xyz="${hand_palm_length/2} 0 0"/>
-    <axis xyz="0 1 0"/>
-    <limit effort="50" lower="0" upper="0.05" velocity="0.4" />
   </joint>
   <!-- Camera -->
@@ -524,24 +520,4 @@
     </actuator>
   </transmission>
-  <transmission name="tran3">
-    <type>transmission_interface/SimpleTransmission</type>
-    <joint name="left_finger_joint">
-      <hardwareInterface>hardware_interface/EffortJointInterface</hardwareInterface>
-    </joint>
-    <actuator name="motor3">
-      <hardwareInterface>hardware_interface/EffortJointInterface</hardwareInterface>
-      <mechanicalReduction>1</mechanicalReduction>
-    </actuator>
-  </transmission>
-  <transmission name="tran4">
-    <type>transmission_interface/SimpleTransmission</type>
-    <joint name="right_finger_joint">
-      <hardwareInterface>hardware_interface/EffortJointInterface</hardwareInterface>
-    </joint>
-    <actuator name="motor4">
-      <hardwareInterface>hardware_interface/EffortJointInterface</hardwareInterface>
-      <mechanicalReduction>1</mechanicalReduction>
-    </actuator>
-  </transmission>
   <gazebo>
     <plugin name="control" filename="libgazebo_ros_control.so"/>
@@ -549,5 +525,5 @@
   <gazebo>
     <plugin name="joint_state_publisher" filename="libgazebo_ros_joint_state_publisher.so">
-      <jointName>hip_joint, shoulder_joint, elbow_joint, wrist_joint, left_finger_joint, right_finger_joint </jointName>
+      <jointName>hip_joint, shoulder_joint, elbow_joint, wrist_joint</jointName>
     </plugin>
   </gazebo>
