Commit message: Changed the world to have walls.Changed dimensios of robot to get to the first can

File: urdf/bookshelf_robot.urdf.xacro (robot description, xacro)
@@ -16,12 +16,12 @@
   <xacro:property name="chassis_mass" value="2.0"/>
   <!-- Wheel links properties -->
-  <xacro:property name="wheel_length" value="0.08" />
+  <xacro:property name="wheel_length" value="0.05" />
   <xacro:property name="wheel_radius" value="0.2" />
   <xacro:property name="wheel_mass" value="0.2" />
   <!-- Caster leg link propersties -->
-  <xacro:property name="caster_leg_length" value="0.05" />
-  <xacro:property name="caster_leg_width" value="0.05" />
+  <xacro:property name="caster_leg_length" value="0.03" />
+  <xacro:property name="caster_leg_width" value="0.03" />
   <xacro:property name="caster_leg_height" value="0.1" />
-  <xacro:property name="caster_leg_mass" value="0.1"/>
+  <xacro:property name="caster_leg_mass" value="0.7"/>
   <!-- Caster leg link properties -->
   <xacro:property name="caster_radius" value="0.04"/>
@@ -44,5 +44,5 @@
   <!-- Elbow properties -->
   <xacro:property name="elbow_radius" value="0.05"/>
-  <xacro:property name="elbow_length" value="0.7"/>
+  <xacro:property name="elbow_length" value="0.8"/>
   <xacro:property name="elbow_mass" value="0.1" />
   <!-- Hand properties -->
@@ -65,5 +65,5 @@
   <xacro:property name="camera_mass" value="0.01" />
   <!-- Laser Scanner -->
-  <xacro:property name="lidar_base_length" value="0.04" />
+  <xacro:property name="lidar_base_length" value="0.02" />
   <xacro:property name="lidar_base_radius" value="0.01" />
   <xacro:property name="lidar_base_mass" value="0.05"/>
@@ -278,5 +278,5 @@
     <origin rpy="0 ${-PI/2} 0" xyz="0 ${-2*arm_radius} ${-torso_length/2}"/>
     <axis xyz="1 0 0"/>
-    <limit effort="100.0" lower="0.0" upper="1.1" velocity="100" />
+    <limit effort="100.0" lower="0.0" upper="1.15" velocity="100" />
   </joint>
   <link name="elbow">
@@ -305,5 +305,5 @@
     <origin rpy="0 0 0" xyz="0 ${2*arm_radius} ${-arm_length/2}"/>
     <axis xyz="0 0 1"/>
-    <limit effort="10.0" lower="0.0" upper="0.25" velocity="10" />
+    <limit effort="10.0" lower="0.0" upper="0.35" velocity="10" />
   </joint>
   <link name="hand_base">
@@ -411,9 +411,9 @@
     <collision>
       <geometry>
-      <box size="${camera_dimensions} ${camera_dimensions} ${camera_dimensions}"/>
-      </geometry>
-    </collision>
-    <visual>
-      <origin xyz="${-camera_dimensions/2} 0 0" rpy="0 0 0"/>
+      <box size="${camera_dimensions} ${2*camera_dimensions} ${camera_dimensions}"/>
+      </geometry>
+    </collision>
+    <visual>
+      <origin xyz="${-camera_dimensions/2} 0 ${-camera_dimensions/2}" rpy="0 0 0"/>
       <geometry>
       <box size="${camera_dimensions} ${camera_dimensions} ${camera_dimensions}"/>
@@ -427,5 +427,5 @@
   </link>
   <joint name="camera_joint" type="fixed">
-    <origin xyz="${-elbow_radius} 0 ${-elbow_length}" rpy="${PI} ${PI/2} 0"/>
+    <origin xyz="${-elbow_radius-0.04} 0 ${-0.9*elbow_length}" rpy="${PI} ${PI/2.5} 0"/>
     <parent link="elbow"/>
     <child link="camera_link"/>

Commit message: Tried to implement move_base. Still not working. Commented in the launch file. everything else seems stable

File: urdf/bookshelf_robot.urdf.xacro (robot description, xacro)
@@ -75,5 +75,5 @@
   <!-- Mobile base implementation -->
   <!-- ########################## -->
-  <link name="footprint">
+  <!-- <link name="footprint">
   </link>
   <joint name="base_joint" type="fixed">
@@ -81,6 +81,6 @@
     <child link="chassis"/>
     <origin rpy="0 0 0" xyz="0 0 ${wheel_radius}"/>
-  </joint>
-  <link name="chassis">
+  </joint> -->
+  <link name="base_link">
     <visual>
       <geometry>
@@ -118,5 +118,5 @@
  <joint name="left_wheel_joint" type="continuous">
     <axis xyz="0 0 1"/>
-    <parent link="chassis"/>
+    <parent link="base_link"/>
     <child link="left_wheel"/>
     <origin rpy="${-PI/2} 0 0" xyz="${-chassis_length/4} ${-chassis_width/2-wheel_length/2} 0}"/>
@@ -141,5 +141,5 @@
   <joint name="right_wheel_joint" type="continuous">
     <axis xyz="0 0 1"/>
-    <parent link="chassis"/>
+    <parent link="base_link"/>
     <child link="right_wheel"/>
     <origin rpy="${-PI/2} 0 0" xyz="${-chassis_length/4}  ${+chassis_width/2+wheel_length/2} 0"/>
@@ -163,5 +163,5 @@
   </link>
   <joint name="chassis_caster_leg_joint" type="fixed">
-    <parent link="chassis"/>
+    <parent link="base_link"/>
     <child link="caster_leg"/>
     <origin rpy="0 0 0" xyz="${3*chassis_length/8} 0 ${-chassis_height/2-caster_leg_height/2}"/>
@@ -194,5 +194,5 @@
       <leftJoint>left_wheel_joint</leftJoint>
       <rightJoint>right_wheel_joint</rightJoint>
-      <robotBaseFrame>chassis</robotBaseFrame>
+      <robotBaseFrame>base_link</robotBaseFrame>
       <wheelSeparation>${chassis_width-wheel_length}</wheelSeparation>
       <wheelDiameter>${2*wheel_radius}</wheelDiameter>
@@ -225,5 +225,5 @@
   </link>
   <joint name="chassis_arm_base" type="fixed">
-    <parent link="chassis"/>
+    <parent link="base_link"/>
     <child link="arm_base"/>
     <origin rpy="${-PI} 0 0" xyz="0 0 ${chassis_height/2+arm_base_length/2}"/>
@@ -454,5 +454,5 @@
   <joint name="base_lidar_joint" type="fixed">
     <origin xyz="${chassis_length/3} 0 ${chassis_height/2}" rpy="0 0 0"/>
-    <parent link="chassis"/>
+    <parent link="base_link"/>
     <child link="lidar_base"/>
   </joint>

Commit message: Add buttons for diffenrent heights

File: urdf/bookshelf_robot.urdf.xacro (robot description, xacro)
@@ -14,17 +14,17 @@
   <xacro:property name="chassis_width" value="0.5" />
   <xacro:property name="chassis_height" value="0.1" />
-  <xacro:property name="chassis_mass" value="2.0"/>
+  <xacro:property name="chassis_mass" value="5.0"/>
   <!-- Wheel links properties -->
-  <xacro:property name="wheel_length" value="0.05" />
+  <xacro:property name="wheel_length" value="0.1" />
   <xacro:property name="wheel_radius" value="0.2" />
-  <xacro:property name="wheel_mass" value="0.2" />
+  <xacro:property name="wheel_mass" value="1" />
   <!-- Caster leg link propersties -->
   <xacro:property name="caster_leg_length" value="0.03" />
   <xacro:property name="caster_leg_width" value="0.03" />
-  <xacro:property name="caster_leg_height" value="0.1" />
-  <xacro:property name="caster_leg_mass" value="0.7"/>
+  <xacro:property name="caster_leg_height" value="0.08" />
+  <xacro:property name="caster_leg_mass" value="1"/>
   <!-- Caster leg link properties -->
   <xacro:property name="caster_radius" value="0.04"/>
-  <xacro:property name="caster_mass" value="0.1"/>
+  <xacro:property name="caster_mass" value="0.5"/>
   <!-- ############ -->
   <!-- Robotic arm  -->
@@ -63,4 +63,5 @@
   <!-- Camera -->
   <xacro:property name="camera_dimensions" value="0.05" />
+  <xacro:property name="camera_gripper_dimensions" value="0.025" />
   <xacro:property name="camera_mass" value="0.01" />
   <!-- Laser Scanner -->
@@ -431,4 +432,27 @@
     <child link="camera_link"/>
   </joint>
+  <link name="camera_gripper_link">
+    <collision>
+      <geometry>
+      <box size="${camera_gripper_dimensions} ${2*camera_gripper_dimensions} ${camera_gripper_dimensions}"/>
+      </geometry>
+    </collision>
+    <visual>
+      <origin xyz="${-camera_gripper_dimensions/2} 0 ${-camera_gripper_dimensions/2}" rpy="0 0 0"/>
+      <geometry>
+      <box size="${camera_gripper_dimensions} ${camera_gripper_dimensions} ${camera_gripper_dimensions}"/>
+      </geometry>
+      <material name="white"/>
+    </visual>
+    <inertial>
+      <mass value="${camera_mass}"/>
+      <box_inertia m="${camera_mass}" x="${camera_gripper_dimensions}" y="${camera_gripper_dimensions}" z="${camera_gripper_dimensions}"/>
+    </inertial>
+  </link>
+  <joint name="camera_gripper_joint" type="fixed">
+    <origin xyz="${-hand_finger_length/2} 0 ${-hand_finger_height/2}" rpy="${PI} 0 ${PI/2}"/>
+    <parent link="hand_right_finger"/>
+    <child link="camera_gripper_link"/>
+  </joint>
   <!-- Laser Scanner -->
 <link name="lidar_base">
@@ -453,5 +477,5 @@
   </link>
   <joint name="base_lidar_joint" type="fixed">
-    <origin xyz="${chassis_length/3} 0 ${chassis_height/2}" rpy="0 0 0"/>
+    <origin xyz="${0.9*chassis_length/2} 0 ${chassis_height/2}" rpy="0 0 0"/>
     <parent link="base_link"/>
     <child link="lidar_base"/>
@@ -462,5 +486,5 @@
         <box size="${lidar_length} ${lidar_width} ${lidar_height}"/>
       </geometry>
-      <origin xyz="0 0 0" rpy="0 0 0"/>
+      <origin xyz="0 0 ${-lidar_height/2}" rpy="0 0 0"/>
       <material name="white"/>
     </visual>
@@ -476,5 +500,5 @@
   </link>
   <joint name="lidar_joint" type="fixed">
-    <origin xyz="0 0 ${lidar_base_length}" rpy="0 0 0"/>
+    <origin xyz="0 0 ${lidar_base_length/2+lidar_height}" rpy="0 0 0"/>
     <parent link="lidar_base"/>
     <child link="lidar_link"/>

Commit message: Wrist joint button added

File: urdf/bookshelf_robot.urdf.xacro (robot description, xacro)
@@ -71,5 +71,5 @@
   <xacro:property name="lidar_length" value="0.05" />
   <xacro:property name="lidar_width" value="0.05" />
-  <xacro:property name="lidar_height" value="0.05" />
+  <xacro:property name="lidar_height" value="0.01" />
   <xacro:property name="lidar_mass" value="0.1"/>
   <!-- ########################## -->
@@ -500,5 +500,5 @@
   </link>
   <joint name="lidar_joint" type="fixed">
-    <origin xyz="0 0 ${lidar_base_length/2+lidar_height}" rpy="0 0 0"/>
+    <origin xyz="0 0 ${lidar_base_length/2+lidar_height}" rpy="0 ${-PI/128} 0"/>
     <parent link="lidar_base"/>
     <child link="lidar_link"/>

Commit message: Added scan interpretation of base position. Hardcoded joints to grap second and third can

File: urdf/bookshelf_robot.urdf.xacro (robot description, xacro)
@@ -22,5 +22,5 @@
   <xacro:property name="caster_leg_length" value="0.03" />
   <xacro:property name="caster_leg_width" value="0.03" />
-  <xacro:property name="caster_leg_height" value="0.08" />
+  <xacro:property name="caster_leg_height" value="0.1" />
   <xacro:property name="caster_leg_mass" value="1"/>
   <!-- Caster leg link properties -->
